File: kicad/board.kicad_pcb (KiCad board)
At the start: 2 copper layers, 100 x 100 mm, 30 parts

Commit message: MCU /  TRRS position update
Parts:
- removed the JP1 at (140.0, 135.5)
- removed the JP2 at (140.0, 135.5)
- moved AudioJack 60.2 mm to (184.1, 127.0), turned to 76 degrees
- moved AudioJack 60.2 mm to (184.1, 126.9), turned to -104 degrees
- moved HOLE5 23.1 mm to (103.4, 111.5)
- moved U? 16.2 mm to (95.7, 127.8), turned to 86 degrees
- moved JP1 11.8 mm to (132.7, 146.4)
- moved JP2 11.8 mm to (132.7, 146.4)
- moved HOLE3 9.07 mm to (179.5, 115.8)
- renumbered JP3 to JP1, JP4 to JP2
Connections:
- AudioJack pad S: Net-(JP2-A) -> GND
- AudioJack pad T: Net-(JP1-A) -> GND
- AudioJack pad S: Net-(JP1-A) -> GND
- AudioJack pad T: Net-(JP2-A) -> GND
Routing:
- net SERIAL: track 0.00 -> 100.6 mm
- net VCC: track 30.6 -> 112.5 mm
- net matrix_pinky_bottom: track 34.7 -> 10.3 mm
- net Net-(JP3-B): track 17.5 -> 40.9 mm
- net thumb_reachy: track 65.9 -> 88.9 mm
- net thumb_tucky: track 54.0 -> 75.5 mm
- net thumb_inner: track 32.5 -> 52.6 mm
- net matrix_pinky_home: track 50.2 -> 31.3 mm
- net matrix_inner_top: track 117.6 -> 134.4 mm
- net matrix_pinky_top: track 66.2 -> 49.7 mm
- net matrix_inner_home: track 101.5 -> 115.4 mm
- net Net-(JP1-A): track 13.1 -> 0.00 mm
- net matrix_inner_bottom: track 74.7 -> 83.7 mm
- net matrix_middle_bottom: track 63.1 -> 55.1 mm
- net Net-(JP2-A): track 7.86 -> 0.00 mm
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Other:
- outline, holes or cut-outs redrawn
